File: eagle/wmBoard1/Rocket3RTC.brd (EAGLE design)
At the start: 42.9 x 67.9 mm, 6 parts

Commit message: Updated for board routing
Parts:
- moved DS3231 1.27 mm to (36.2, 15.2)
- moved MPL3115A2 1.27 mm to (36.2, 36.8)
- moved BNO055-1 1.27 mm to (8.26, 17.8)
- moved BNO055-2 1.27 mm to (8.26, 45.7)
Routing:
- net VBAT: track 69.9 -> 82.9 mm
- net GND: track 86.6 -> 96.3 mm
- net SCL: track 84.1 -> 91.8 mm
- net SDA: track 82.4 -> 86.2 mm
- net +3V3: track 28.1 -> 29.4 mm
- net D11: track 6.13 -> 6.66 mm
Other:
- board text added: "If found please call (206) 790-7989"
