File: eagle/wmBoard2/Rocket4Narrow.brd (EAGLE design)
At the start: 24.4 x 78.1 mm, 4 parts

Commit message: Updated for board routing
Routing:
- net SCL: track 71.9 -> 73.3 mm
- net SDA: track 78.0 -> 79.1 mm
- net D11: track 42.8 -> 43.5 mm
Other:
- board text added: "If found please call (206) 790-7989"
Changed lines of the file:
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@@
 <setting verticaltext="up"/>
 </settings>
-<grid distance="0.01" unitdist="inch" unit="mil" style="lines" multiple="1" display="yes" altdistance="5" altunitdist="mil" altunit="mil"/>
+<grid distance="2" unitdist="mil" unit="mil" style="lines" multiple="1" display="yes" altdistance="5" altunitdist="mil" altunit="mil"/>
 <layers>
 <layer number="1" name="Top" color="4" fill="1" visible="yes" active="yes"/>
@@
 <layer number="18" name="Vias" color="2" fill="1" visible="yes" active="yes"/>
 <layer number="19" name="Unrouted" color="6" fill="1" visible="no" active="yes"/>
-<layer number="20" name="Dimension" color="24" fill="1" visible="yes" active="yes"/>
+<layer number="20" name="Dimension" color="24" fill="1" visible="no" active="yes"/>
 <layer number="21" name="tPlace" color="7" fill="1" visible="yes" active="yes"/>
-<layer number="22" name="bPlace" color="7" fill="1" visible="no" active="yes"/>
-<layer number="23" name="tOrigins" color="15" fill="1" visible="yes" active="yes"/>
+<layer number="22" name="bPlace" color="7" fill="1" visible="yes" active="yes"/>
+<layer number="23" name="tOrigins" color="15" fill="1" visible="no" active="yes"/>
 <layer number="24" name="bOrigins" color="15" fill="1" visible="no" active="yes"/>
-<layer number="25" name="tNames" color="7" fill="1" visible="yes" active="yes"/>
+<layer number="25" name="tNames" color="7" fill="1" visible="no" active="yes"/>
 <layer number="26" name="bNames" color="7" fill="1" visible="no" active="yes"/>
-<layer number="27" name="tValues" color="7" fill="1" visible="yes" active="yes"/>
+<layer number="27" name="tValues" color="7" fill="1" visible="no" active="yes"/>
 <layer number="28" name="bValues" color="7" fill="1" visible="no" active="yes"/>
 <layer number="29" name="tStop" color="7" fill="3" visible="no" active="yes"/>
@@
 <wire x1="5.715" y1="76.835" x2="5.715" y2="52.07" width="0.1524" layer="21"/>
 <wire x1="5.715" y1="52.07" x2="8.255" y2="52.07" width="0.1524" layer="21"/>
+<text x="15.1892" y="43.8912" size="1.778" layer="22" font="vector" ratio="12" rot="MR270">If found please call
+   (206) 790-7989</text>
 </plain>
 <attributes>
@@
 <contactref element="JP1" pad="13"/>
 <contactref element="JP1" pad="1"/>
+<wire x1="7.03595" y1="55.9331" x2="7.59475" y2="55.9331" width="0.381" layer="16"/>
 <wire x1="7.59475" y1="55.9331" x2="17.06585" y2="55.9331" width="0.381" layer="16"/>
-<wire x1="5.62905" y1="57.8988" x2="7.59475" y2="55.9331" width="0.381" layer="16"/>
-<wire x1="5.62905" y1="64.6894" x2="5.62905" y2="57.8988" width="0.381" layer="16"/>
+<wire x1="5.62905" y1="57.34" x2="7.03595" y2="55.9331" width="0.381" layer="16"/>
+<wire x1="5.62905" y1="64.6894" x2="5.62905" y2="57.34" width="0.381" layer="16"/>
 <wire x1="6.9693" y1="66.02965" x2="5.62905" y2="64.6894" width="0.381" layer="16"/>
 <wire x1="17.06585" y1="55.9331" x2="17.145" y2="55.88" width="0.381" layer="16"/>
@@
 <contactref element="JP3" pad="6"/>
 <contactref element="MPL3115A2" pad="4"/>
-<wire x1="22.225" y1="20.32" x2="22.0881" y2="20.32" width="0.1524" layer="16"/>
-<wire x1="22.0881" y1="20.32" x2="18.57075" y2="23.83735" width="0.1524" layer="16"/>
-<wire x1="18.57075" y1="59.52115" x2="18.57075" y2="23.83735" width="0.1524" layer="16"/>
+<wire x1="22.225" y1="20.32" x2="20.9197" y2="20.32" width="0.1524" layer="16"/>
+<wire x1="20.9197" y1="20.32" x2="18.57075" y2="22.66895" width="0.1524" layer="16"/>
+<wire x1="18.57075" y1="59.52115" x2="18.57075" y2="22.66895" width="0.1524" layer="16"/>
 <wire x1="17.1552" y1="60.9367" x2="18.57075" y2="59.52115" width="0.1524" layer="16"/>
 <wire x1="17.1552" y1="60.9367" x2="17.145" y2="60.96" width="0.1524" layer="16"/>
@@
 <contactref element="MPL3115A2" pad="6"/>
 <contactref element="BNO055-1" pad="5"/>
-<wire x1="8.2202" y1="21.6227" x2="22.225" y2="7.62" width="0.1524" layer="1"/>
-<wire x1="8.2202" y1="59.77515" x2="8.2202" y2="21.6227" width="0.1524" layer="1"/>
+<wire x1="19.837284375" y1="7.62" x2="22.225" y2="7.62" width="0.1524" layer="1"/>
+<wire x1="19.837284375" y1="7.62" x2="8.2202" y2="19.23534375" width="0.1524" layer="1"/>
+<wire x1="8.2202" y1="59.77515" x2="8.2202" y2="19.23534375" width="0.1524" layer="1"/>
 <wire x1="7.05865" y1="60.9367" x2="8.2202" y2="59.77515" width="0.1524" layer="1"/>
 <wire x1="7.05865" y1="60.9367" x2="6.985" y2="60.96" width="0.1524" layer="1"/>
@@
 <contactref element="MPL3115A2" pad="7"/>
 <contactref element="BNO055-1" pad="4"/>
-<wire x1="22.1386" y1="5.334" x2="22.1386" y2="5.1664" width="0.1524" layer="1"/>
-<wire x1="22.225" y1="5.08" x2="22.1386" y2="5.1664" width="0.1524" layer="1"/>
-<wire x1="22.1386" y1="5.334" x2="5.80775" y2="21.66485" width="0.1524" layer="1"/>
-<wire x1="5.80775" y1="62.27695" x2="5.80775" y2="21.66485" width="0.1524" layer="1"/>
-<wire x1="6.9693" y1="63.4385" x2="5.80775" y2="62.27695" width="0.1524" layer="1"/>
+<wire x1="22.225" y1="5.08" x2="20.3454" y2="5.08" width="0.1524" layer="1"/>
+<wire x1="20.3454" y1="5.08" x2="5.70615" y2="19.71925" width="0.1524" layer="1"/>
+<wire x1="5.70615" y1="62.17535" x2="5.70615" y2="19.71925" width="0.1524" layer="1"/>
+<wire x1="6.9693" y1="63.4385" x2="5.70615" y2="62.17535" width="0.1524" layer="1"/>
 <wire x1="6.9693" y1="63.4385" x2="6.985" y2="63.5" width="0.1524" layer="1"/>
 <wire x1="12.06225" y1="68.53145" x2="17.06585" y2="68.53145" width="0.1524" layer="16"/>
@@
 </board>
 </drawing>
+<compatibility>
+<note version="6.3" minversion="6.2.2" severity="warning">
+Since Version 6.2.2 text objects can contain more than one line,
+which will not be processed correctly with this version.
+</note>
+</compatibility>
 </eagle>
